Commit message: fixes to hokuyo and velodyne parameters

File: uol_cmp9767m_base/urdf/sensors.xacro (robot description, xacro)
@@ -23,5 +23,5 @@
     </inertial>
   </link>
-   <joint name="base_link_hokuyo" type="fixed">
+  <joint name="$(arg robot_name)_base_link_hokuyo" type="fixed">
     <parent link="$(arg tf_prefix)/base_link"/>
     <child link="$(arg tf_prefix)/hokuyo"/>
@@ -31,5 +31,5 @@
   <!--hokuyo-->
   <gazebo reference="$(arg tf_prefix)/hokuyo">
-    <sensor name="$(arg robot_name)_head_hokuyo_sensor" type="ray">
+    <sensor name="$(arg robot_name)hokuyo_sensor" type="ray">
       <pose>0 0 0 0 0 0</pose>
       <visualize>true</visualize>
@@ -60,6 +60,6 @@
         </noise>
       </ray>
-      <plugin name="$(arg robot_name)_hokuyo_node" filename="libgazebo_ros_laser.so">
-        <topicName>hokuyo_scan</topicName>
+      <plugin name="$(arg robot_name)hokuyo_node" filename="libgazebo_ros_laser.so">
+        <topicName>scan</topicName>
         <frameName>hokuyo</frameName>
       </plugin>
@@ -68,5 +68,5 @@
   <!-- Velodyne VLP16 -->
   <xacro:include filename="$(find velodyne_description)/urdf/VLP-16.urdf.xacro"/>
-  <VLP-16 parent="/base_link" name="/velodyne" topic="/velodyne_points" hz="10" samples="440" min_range="0.9"  max_range="130.0" noise="0.008">
+  <VLP-16 parent="$(arg tf_prefix)/base_link" name="$(arg tf_prefix)/velodyne" topic="$(arg robot_name)/velodyne_points" hz="10" samples="440" min_range="0.9"  max_range="130.0" noise="0.008">
     <origin xyz="0 0 1.56" rpy="0 0 0" />
   </VLP-16>

Commit message: Added the kinect processor node: It subscribes to the kinect sensor topics and published its own topics after finding weeds in the image

File: uol_cmp9767m_base/urdf/sensors.xacro (robot description, xacro)
@@ -248,7 +248,7 @@
   <xacro:property name="kinect2_cam_py" value="0.0" />
   <xacro:property name="kinect2_cam_pz" value="0.5" />
-  <xacro:property name="kinect2_cam_or" value="0.0" />
-  <xacro:property name="kinect2_cam_op" value="${M_PI/2}" />
-  <xacro:property name="kinect2_cam_oy" value="-${M_PI/2}" />
+  <xacro:property name="kinect2_cam_or" value="-${M_PI/2}" />
+  <xacro:property name="kinect2_cam_op" value="${M_PI/4}" />
+  <xacro:property name="kinect2_cam_oy" value="0.0" />
   <link name="$(arg tf_prefix)/${kinect2_name}_link">
     <visual>

Commit message: Camera Orientation Changed

File: uol_cmp9767m_base/urdf/sensors.xacro (robot description, xacro)
@@ -248,7 +248,7 @@
   <xacro:property name="kinect2_cam_py" value="0.0" />
   <xacro:property name="kinect2_cam_pz" value="0.5" />
-  <xacro:property name="kinect2_cam_or" value="0.0" />
-  <xacro:property name="kinect2_cam_op" value="${M_PI/2}" />
-  <xacro:property name="kinect2_cam_oy" value="-${M_PI/2}" />
+  <xacro:property name="kinect2_cam_or" value="0" />
+  <xacro:property name="kinect2_cam_op" value="${M_PI/4}" />
+  <xacro:property name="kinect2_cam_oy" value="-${2*M_PI}" />
   <link name="$(arg tf_prefix)/${kinect2_name}_link">
     <visual>

Commit message: init commit after errors

File: uol_cmp9767m_base/urdf/sensors.xacro (robot description, xacro)
@@ -248,7 +248,7 @@
   <xacro:property name="kinect2_cam_py" value="0.0" />
   <xacro:property name="kinect2_cam_pz" value="0.5" />
-  <xacro:property name="kinect2_cam_or" value="0.0" />
-  <xacro:property name="kinect2_cam_op" value="${M_PI/2}" />
-  <xacro:property name="kinect2_cam_oy" value="-${M_PI/2}" />
+  <xacro:property name="kinect2_cam_or" value="${M_PI/2}" /> <!-- change ${M_PI/2}-->
+  <xacro:property name="kinect2_cam_op" value="${M_PI/4.3}" />
+  <xacro:property name="kinect2_cam_oy" value="0" />
   <link name="$(arg tf_prefix)/${kinect2_name}_link">
     <visual>

Commit message: Re-oriented camera to original position for greater accuracy in image processing

File: uol_cmp9767m_base/urdf/sensors.xacro (robot description, xacro)
@@ -249,6 +249,6 @@
   <xacro:property name="kinect2_cam_pz" value="0.5" />
   <xacro:property name="kinect2_cam_or" value="0" />
-  <xacro:property name="kinect2_cam_op" value="${M_PI/4}" />
-  <xacro:property name="kinect2_cam_oy" value="-${2*M_PI}" />
+  <xacro:property name="kinect2_cam_op" value="${M_PI/2}" />
+  <xacro:property name="kinect2_cam_oy" value="-${M_PI/2}" />
   <link name="$(arg tf_prefix)/${kinect2_name}_link">
     <visual>

Commit message: student submission

File: uol_cmp9767m_base/urdf/sensors.xacro (robot description, xacro)
@@ -248,7 +248,7 @@
   <xacro:property name="kinect2_cam_py" value="0.0" />
   <xacro:property name="kinect2_cam_pz" value="0.5" />
-  <xacro:property name="kinect2_cam_or" value="0.0" />
-  <xacro:property name="kinect2_cam_op" value="${M_PI/2}" />
-  <xacro:property name="kinect2_cam_oy" value="-${M_PI/2}" />
+  <xacro:property name="kinect2_cam_or" value="${M_PI/2}" />
+  <xacro:property name="kinect2_cam_op" value="${M_PI/2.25}" />
+  <xacro:property name="kinect2_cam_oy" value="0.0" />
   <link name="$(arg tf_prefix)/${kinect2_name}_link">
     <visual>
@@ -279,5 +279,5 @@
     <parent link="$(arg tf_prefix)/${kinect2_name}_link"/>
     <child link="$(arg tf_prefix)/${kinect2_name}_rgb_optical_frame"/>
-    <origin xyz="0 0.0125 0.016" rpy="-1.57 0 -1.57"/>
+    <origin xyz="0 0.0125 0.016" rpy="-1.57 0 -1.13"/>
   </joint>
   <link name="$(arg tf_prefix)/${kinect2_name}_depth_optical_frame"/>

Commit message: fixed meshes for melodic

File: uol_cmp9767m_base/urdf/sensors.xacro (robot description, xacro)
@@ -126,10 +126,10 @@
     <visual>
       <geometry>
-        <mesh filename="package://velodyne_description8/meshes/VLP16_base_1.dae" />
-      </geometry>
-    </visual>
-    <visual>
-      <geometry>
-        <mesh filename="package://velodyne_description8/meshes/VLP16_base_2.dae" />
+        <mesh filename="package://velodyne_description/meshes/VLP16_base_1.dae" />
+      </geometry>
+    </visual>
+    <visual>
+      <geometry>
+        <mesh filename="package://velodyne_description/meshes/VLP16_base_2.dae" />
       </geometry>
     </visual>
@@ -155,5 +155,5 @@
       <origin xyz="0 0 -0.0377" />
       <geometry>
-        <mesh filename="package://velodyne_description8/meshes/VLP16_scan.dae" />
+        <mesh filename="package://velodyne_description/meshes/VLP16_scan.dae" />
       </geometry>
     </visual>
@@ -254,5 +254,5 @@
     <visual>
       <geometry>
-        <mesh filename="package://kinect2_description/meshes/sensors/kinect2.dae"/>
+        <!-- DISABLE for NOW: <mesh filename="package://kinect2_description/meshes/sensors/kinect2.dae"/>-->
       </geometry>
       <origin xyz="0.02 0 0" rpy="0 0 3.141592"/>

Commit message: thorvald tf_prefix must have a / at tail end

File: uol_cmp9767m_base/urdf/sensors.xacro (robot description, xacro)
@@ -4,5 +4,5 @@
   <xacro:arg name="tf_prefix" default=""/>
   <!-- Fake Sprayer Laser -->
-  <link name="$(arg tf_prefix)/sprayer">
+  <link name="$(arg tf_prefix)sprayer">
     <collision>
       <origin xyz="0 0 0" rpy="0 0 0"/>
@@ -21,15 +21,15 @@
     </inertial>
   </link>
-  <gazebo reference="$(arg tf_prefix)/sprayer">
+  <gazebo reference="$(arg tf_prefix)sprayer">
     <material>Gazebo/Orange</material>
   </gazebo>
   <joint name="$(arg robot_name)_base_link_sprayer" type="fixed">
-    <parent link="$(arg tf_prefix)/base_link"/>
-    <child link="$(arg tf_prefix)/sprayer"/>
+    <parent link="$(arg tf_prefix)base_link"/>
+    <child link="$(arg tf_prefix)sprayer"/>
     <axis xyz="1 0 0" />
     <origin xyz="-0.45 0.000 0.5" rpy="0 0 0"/>
   </joint>
   <!-- Hokuyo Laser -->
-  <link name="$(arg tf_prefix)/hokuyo">
+  <link name="$(arg tf_prefix)hokuyo">
     <collision>
       <origin xyz="0 0 0" rpy="0 0 0"/>
@@ -51,11 +51,11 @@
   </link>
   <joint name="$(arg robot_name)_base_link_hokuyo" type="fixed">
-    <parent link="$(arg tf_prefix)/base_link"/>
-    <child link="$(arg tf_prefix)/hokuyo"/>
+    <parent link="$(arg tf_prefix)base_link"/>
+    <child link="$(arg tf_prefix)hokuyo"/>
     <axis xyz="0 1 0" />
     <origin xyz="0.7025 0.005 0.66" rpy="0 0 0"/>
   </joint>
   <!--hokuyo-->
-  <gazebo reference="$(arg tf_prefix)/hokuyo">
+  <gazebo reference="$(arg tf_prefix)hokuyo">
     <sensor name="$(arg robot_name)hokuyo_sensor" type="ray">
       <pose>0 0 0 0 0 0</pose>
@@ -113,8 +113,8 @@
   <joint name="$(arg robot_name)_${velodyne_name}_base_mount_joint" type="fixed">
     <xacro:insert_block name="velodyne_origin" />
-    <parent link="$(arg tf_prefix)/${velodyne_parent}"/>
-    <child link="$(arg tf_prefix)/${velodyne_name}_link"/>
-  </joint>
-  <link name="$(arg tf_prefix)/${velodyne_name}_link">
+    <parent link="$(arg tf_prefix)${velodyne_parent}"/>
+    <child link="$(arg tf_prefix)${velodyne_name}_link"/>
+  </joint>
+  <link name="$(arg tf_prefix)${velodyne_name}_link">
     <inertial>
       <mass value="0.83"/>
@@ -143,8 +143,8 @@
   <joint name="$(arg robot_name)_${velodyne_name}_base_scan_joint" type="fixed" >
     <origin xyz="0 0 0.0377" rpy="0 0 0" />
-    <parent link="$(arg tf_prefix)/${velodyne_name}_link" />
-    <child link="$(arg tf_prefix)/${velodyne_name}"/>
-  </joint>
-  <link name="$(arg tf_prefix)/${velodyne_name}">
+    <parent link="$(arg tf_prefix)${velodyne_name}_link" />
+    <child link="$(arg tf_prefix)${velodyne_name}"/>
+  </joint>
+  <link name="$(arg tf_prefix)${velodyne_name}">
     <inertial>
       <mass value="0.01"/>
@@ -160,5 +160,5 @@
   </link>
   <!-- Gazebo requires the velodyne_gazebo_plugins package -->
-  <gazebo reference="$(arg tf_prefix)/${velodyne_name}">
+  <gazebo reference="$(arg tf_prefix)${velodyne_name}">
     <xacro:if value="${velodyne_gpu}">
       <sensor type="gpu_ray" name="$(arg robot_name)_${velodyne_name}-VLP16">
@@ -251,5 +251,5 @@
   <xacro:property name="kinect2_cam_op" value="${M_PI/2}" />
   <xacro:property name="kinect2_cam_oy" value="-${M_PI/2}" />
-  <link name="$(arg tf_prefix)/${kinect2_name}_link">
+  <link name="$(arg tf_prefix)${kinect2_name}_link">
     <visual>
       <geometry>
@@ -271,21 +271,21 @@
   </link>
   <joint name="$(arg robot_name)_${kinect2_name}_joint" type="fixed">
-    <parent link="$(arg tf_prefix)/${kinect2_parent}"/>
-    <child link="$(arg tf_prefix)/${kinect2_name}_link"/>
+    <parent link="$(arg tf_prefix)${kinect2_parent}"/>
+    <child link="$(arg tf_prefix)${kinect2_name}_link"/>
     <origin xyz="${kinect2_cam_px} ${kinect2_cam_py} ${kinect2_cam_pz}" rpy="${kinect2_cam_or} ${kinect2_cam_op} ${kinect2_cam_oy}"/>
   </joint>
-  <link name="$(arg tf_prefix)/${kinect2_name}_rgb_optical_frame"/>
+  <link name="$(arg tf_prefix)${kinect2_name}_rgb_optical_frame"/>
   <joint name="$(arg robot_name)_${kinect2_name}_rgb_joint" type="fixed">
-    <parent link="$(arg tf_prefix)/${kinect2_name}_link"/>
-    <child link="$(arg tf_prefix)/${kinect2_name}_rgb_optical_frame"/>
+    <parent link="$(arg tf_prefix)${kinect2_name}_link"/>
+    <child link="$(arg tf_prefix)${kinect2_name}_rgb_optical_frame"/>
     <origin xyz="0 0.0125 0.016" rpy="-1.57 0 -1.57"/>
   </joint>
-  <link name="$(arg tf_prefix)/${kinect2_name}_depth_optical_frame"/>
+  <link name="$(arg tf_prefix)${kinect2_name}_depth_optical_frame"/>
   <joint name="$(arg robot_name)_${kinect2_name}_depth_joint" type="fixed">
-    <parent link="$(arg tf_prefix)/${kinect2_name}_link"/>
-    <child link="$(arg tf_prefix)/${kinect2_name}_depth_optical_frame"/>
+    <parent link="$(arg tf_prefix)${kinect2_name}_link"/>
+    <child link="$(arg tf_prefix)${kinect2_name}_depth_optical_frame"/>
     <origin xyz="0 -0.0125 0.016" rpy="-1.57 0 -1.57"/>
   </joint>
-  <gazebo reference="$(arg tf_prefix)/${kinect2_name}_link">
+  <gazebo reference="$(arg tf_prefix)${kinect2_name}_link">
     <sensor name="$(arg robot_name)_${kinect2_name}_sensor" type="depth">
       <always_on>true</always_on>
@@ -333,5 +333,5 @@
     </sensor>
   </gazebo>
-  <gazebo reference="$(arg tf_prefix)/${kinect2_name}_link">
+  <gazebo reference="$(arg tf_prefix)${kinect2_name}_link">
     <sensor name="$(arg robot_name)_${kinect2_name}_camera" type="camera">
       <always_on>true</always_on>

Commit message: re-enabling kinect2

File: uol_cmp9767m_base/urdf/sensors.xacro (robot description, xacro)
@@ -254,5 +254,5 @@
     <visual>
       <geometry>
-        <!-- DISABLE for NOW: <mesh filename="package://kinect2_description/meshes/sensors/kinect2.dae"/>-->
+        <mesh filename="package://kinect2_description/meshes/sensors/kinect2.dae"/>
       </geometry>
       <origin xyz="0.02 0 0" rpy="0 0 3.141592"/>

Commit message: thorvald tf_prefix must have a / at tail end (#51)
* thorvald tf_prefix must have a / at tail end

* gazebo model hook fix

* re-enabling kinect2

File: uol_cmp9767m_base/urdf/sensors.xacro (robot description, xacro)
@@ -4,5 +4,5 @@
   <xacro:arg name="tf_prefix" default=""/>
   <!-- Fake Sprayer Laser -->
-  <link name="$(arg tf_prefix)/sprayer">
+  <link name="$(arg tf_prefix)sprayer">
     <collision>
       <origin xyz="0 0 0" rpy="0 0 0"/>
@@ -21,15 +21,15 @@
     </inertial>
   </link>
-  <gazebo reference="$(arg tf_prefix)/sprayer">
+  <gazebo reference="$(arg tf_prefix)sprayer">
     <material>Gazebo/Orange</material>
   </gazebo>
   <joint name="$(arg robot_name)_base_link_sprayer" type="fixed">
-    <parent link="$(arg tf_prefix)/base_link"/>
-    <child link="$(arg tf_prefix)/sprayer"/>
+    <parent link="$(arg tf_prefix)base_link"/>
+    <child link="$(arg tf_prefix)sprayer"/>
     <axis xyz="1 0 0" />
     <origin xyz="-0.45 0.000 0.5" rpy="0 0 0"/>
   </joint>
   <!-- Hokuyo Laser -->
-  <link name="$(arg tf_prefix)/hokuyo">
+  <link name="$(arg tf_prefix)hokuyo">
     <collision>
       <origin xyz="0 0 0" rpy="0 0 0"/>
@@ -51,11 +51,11 @@
   </link>
   <joint name="$(arg robot_name)_base_link_hokuyo" type="fixed">
-    <parent link="$(arg tf_prefix)/base_link"/>
-    <child link="$(arg tf_prefix)/hokuyo"/>
+    <parent link="$(arg tf_prefix)base_link"/>
+    <child link="$(arg tf_prefix)hokuyo"/>
     <axis xyz="0 1 0" />
     <origin xyz="0.7025 0.005 0.66" rpy="0 0 0"/>
   </joint>
   <!--hokuyo-->
-  <gazebo reference="$(arg tf_prefix)/hokuyo">
+  <gazebo reference="$(arg tf_prefix)hokuyo">
     <sensor name="$(arg robot_name)hokuyo_sensor" type="ray">
       <pose>0 0 0 0 0 0</pose>
@@ -113,8 +113,8 @@
   <joint name="$(arg robot_name)_${velodyne_name}_base_mount_joint" type="fixed">
     <xacro:insert_block name="velodyne_origin" />
-    <parent link="$(arg tf_prefix)/${velodyne_parent}"/>
-    <child link="$(arg tf_prefix)/${velodyne_name}_link"/>
-  </joint>
-  <link name="$(arg tf_prefix)/${velodyne_name}_link">
+    <parent link="$(arg tf_prefix)${velodyne_parent}"/>
+    <child link="$(arg tf_prefix)${velodyne_name}_link"/>
+  </joint>
+  <link name="$(arg tf_prefix)${velodyne_name}_link">
     <inertial>
       <mass value="0.83"/>
@@ -143,8 +143,8 @@
   <joint name="$(arg robot_name)_${velodyne_name}_base_scan_joint" type="fixed" >
     <origin xyz="0 0 0.0377" rpy="0 0 0" />
-    <parent link="$(arg tf_prefix)/${velodyne_name}_link" />
-    <child link="$(arg tf_prefix)/${velodyne_name}"/>
-  </joint>
-  <link name="$(arg tf_prefix)/${velodyne_name}">
+    <parent link="$(arg tf_prefix)${velodyne_name}_link" />
+    <child link="$(arg tf_prefix)${velodyne_name}"/>
+  </joint>
+  <link name="$(arg tf_prefix)${velodyne_name}">
     <inertial>
       <mass value="0.01"/>
@@ -160,5 +160,5 @@
   </link>
   <!-- Gazebo requires the velodyne_gazebo_plugins package -->
-  <gazebo reference="$(arg tf_prefix)/${velodyne_name}">
+  <gazebo reference="$(arg tf_prefix)${velodyne_name}">
     <xacro:if value="${velodyne_gpu}">
       <sensor type="gpu_ray" name="$(arg robot_name)_${velodyne_name}-VLP16">
@@ -251,8 +251,8 @@
   <xacro:property name="kinect2_cam_op" value="${M_PI/2}" />
   <xacro:property name="kinect2_cam_oy" value="-${M_PI/2}" />
-  <link name="$(arg tf_prefix)/${kinect2_name}_link">
-    <visual>
-      <geometry>
-        <!-- DISABLE for NOW: <mesh filename="package://kinect2_description/meshes/sensors/kinect2.dae"/>-->
+  <link name="$(arg tf_prefix)${kinect2_name}_link">
+    <visual>
+      <geometry>
+        <mesh filename="package://kinect2_description/meshes/sensors/kinect2.dae"/>
       </geometry>
       <origin xyz="0.02 0 0" rpy="0 0 3.141592"/>
@@ -271,21 +271,21 @@
   </link>
   <joint name="$(arg robot_name)_${kinect2_name}_joint" type="fixed">
-    <parent link="$(arg tf_prefix)/${kinect2_parent}"/>
-    <child link="$(arg tf_prefix)/${kinect2_name}_link"/>
+    <parent link="$(arg tf_prefix)${kinect2_parent}"/>
+    <child link="$(arg tf_prefix)${kinect2_name}_link"/>
     <origin xyz="${kinect2_cam_px} ${kinect2_cam_py} ${kinect2_cam_pz}" rpy="${kinect2_cam_or} ${kinect2_cam_op} ${kinect2_cam_oy}"/>
   </joint>
-  <link name="$(arg tf_prefix)/${kinect2_name}_rgb_optical_frame"/>
+  <link name="$(arg tf_prefix)${kinect2_name}_rgb_optical_frame"/>
   <joint name="$(arg robot_name)_${kinect2_name}_rgb_joint" type="fixed">
-    <parent link="$(arg tf_prefix)/${kinect2_name}_link"/>
-    <child link="$(arg tf_prefix)/${kinect2_name}_rgb_optical_frame"/>
+    <parent link="$(arg tf_prefix)${kinect2_name}_link"/>
+    <child link="$(arg tf_prefix)${kinect2_name}_rgb_optical_frame"/>
     <origin xyz="0 0.0125 0.016" rpy="-1.57 0 -1.57"/>
   </joint>
-  <link name="$(arg tf_prefix)/${kinect2_name}_depth_optical_frame"/>
+  <link name="$(arg tf_prefix)${kinect2_name}_depth_optical_frame"/>
   <joint name="$(arg robot_name)_${kinect2_name}_depth_joint" type="fixed">
-    <parent link="$(arg tf_prefix)/${kinect2_name}_link"/>
-    <child link="$(arg tf_prefix)/${kinect2_name}_depth_optical_frame"/>
+    <parent link="$(arg tf_prefix)${kinect2_name}_link"/>
+    <child link="$(arg tf_prefix)${kinect2_name}_depth_optical_frame"/>
     <origin xyz="0 -0.0125 0.016" rpy="-1.57 0 -1.57"/>
   </joint>
-  <gazebo reference="$(arg tf_prefix)/${kinect2_name}_link">
+  <gazebo reference="$(arg tf_prefix)${kinect2_name}_link">
     <sensor name="$(arg robot_name)_${kinect2_name}_sensor" type="depth">
       <always_on>true</always_on>
@@ -333,5 +333,5 @@
     </sensor>
   </gazebo>
-  <gazebo reference="$(arg tf_prefix)/${kinect2_name}_link">
+  <gazebo reference="$(arg tf_prefix)${kinect2_name}_link">
     <sensor name="$(arg robot_name)_${kinect2_name}_camera" type="camera">
       <always_on>true</always_on>
